File: Hardware/Eagle/odin_mod.sch (EAGLE design)
At the start: 44 parts, among them Q1 IRLML0030, Q2 IRLML0030, Q3 IRLML0030, Q4 IRLML0030

Commit message: Lowered segment resistors and optimized traces.
Parts:
- R2, R3, R4, R5, R6, R7, R8: value 82 -> 75
Other:
- note added: "If using a photo diode, instead of the vintage LDR, use 6,8 k instead of 47 k. Connect the anode to LIGHTOUT. Actually some LDRs give you different outputs. So, you might lower the resistor value down from 47k to 10 k."
- note removed: "If using a photo diode, instead of the vintage LDR, use 6,8 k instead of 47 k. Connect the anode to LIGHTOUT. Actually some LDR give you different output. So you might change the resistor value down to 10 k."
Changed lines of the file:
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@@
 <part name="SUPPLY2" library="supply2" deviceset="GND" device=""/>
 <part name="SUPPLY3" library="supply2" deviceset="GND" device=""/>
-<part name="R2" library="resistor" deviceset="R-EU_" device="R0402" value="82"/>
-<part name="R3" library="resistor" deviceset="R-EU_" device="R0402" value="82"/>
-<part name="R4" library="resistor" deviceset="R-EU_" device="R0402" value="82"/>
-<part name="R5" library="resistor" deviceset="R-EU_" device="R0402" value="82"/>
-<part name="R6" library="resistor" deviceset="R-EU_" device="R0402" value="82"/>
-<part name="R7" library="resistor" deviceset="R-EU_" device="R0402" value="82"/>
-<part name="R8" library="resistor" deviceset="R-EU_" device="R0402" value="82"/>
+<part name="R2" library="resistor" deviceset="R-EU_" device="R0402" value="75"/>
+<part name="R3" library="resistor" deviceset="R-EU_" device="R0402" value="75"/>
+<part name="R4" library="resistor" deviceset="R-EU_" device="R0402" value="75"/>
+<part name="R5" library="resistor" deviceset="R-EU_" device="R0402" value="75"/>
+<part name="R6" library="resistor" deviceset="R-EU_" device="R0402" value="75"/>
+<part name="R7" library="resistor" deviceset="R-EU_" device="R0402" value="75"/>
+<part name="R8" library="resistor" deviceset="R-EU_" device="R0402" value="75"/>
 <part name="R14" library="resistor" deviceset="R-EU_" device="R0402" value="4.7k"/>
 <part name="R15" library="resistor" deviceset="R-EU_" device="R0402" value="4.7k"/>
@@
 This is public domain.</text>
 <text x="-22.86" y="-110.49" size="2.54" layer="94" font="vector">Pulsar P3 Odin Mk II</text>
-<text x="-45.72" y="27.94" size="1.778" layer="94">If using a photo diode, instead of the vintage
+<text x="-50.038" y="28.956" size="1.778" layer="94">If using a photo diode, instead of the vintage
 LDR, use 6,8 k instead of 47 k. Connect the
-anode to LIGHTOUT. Actually some LDR give
-you different output. So you might change
-the resistor value down to 10 k.</text>
+anode to LIGHTOUT. Actually some LDRs give
+you different outputs. So, you might lower
+the resistor value down from 47k to 10 k.</text>
 <text x="-120.904" y="87.122" size="1.778" layer="94">Do not use
 less than
